Commit message: Skip water mesh in inspection world

File: cpr_inspection_gazebo/urdf/inspection_geometry.urdf.xacro (robot description, xacro)
@@ -13,10 +13,10 @@
       </geometry>
     </visual>
-    <visual>
+    <!-- <visual>
       <origin xyz="0 0 0" rpy="0 0 0"/>
       <geometry>
         <mesh filename="package://cpr_inspection_gazebo/meshes/inspection_water.dae"/>
       </geometry>
-    </visual>
+    </visual> -->
     <collision>
       <origin xyz="0 0 0" rpy="0 0 0"/>
